File: gigasound-hw/gigasound-hw.kicad_pcb (KiCad board)
At the start: 2 copper layers, 115 parts, among them J1 Conn_01x04_Socket, J2 Conn_01x05_Socket, J3 Conn_01x05_Socket, J4 USB_C_Receptacle_USB2.0_16P, J5 PIN_LED_OUT, SW1 PLAY, SW2 Reset, SW4 STOP, SW5 MODE, U1 STM32F401RETx, U5 AMS1117-3.3, Y1 12MHz

Commit message: hw: Finished footprints
Parts:
- removed J3: Conn_01x05_Socket, Connector_PinHeader_2.54mm:PinHeader_1x04_P2.54mm_Vertical
- added J6: Conn_01x04_Socket_OLED, gigalibrary:PinSocket_1x04_P2.54mm_Vertical_OLED_0.96inch, F.Cu at (147.5, 39.5)
- J1: value Conn_01x04_Socket -> Conn_01x05_Socket_FPC_Joycon; footprint Connector_PinHeader_2.54mm:PinHeader_1x04_P2.54mm_Vertical -> gigalibrary:Joycon-FPC-1x05-P0.5mm
- J2: value Conn_01x05_Socket -> Conn_01x05_Socket_UART; footprint gigalibrary:Joycon-FPC-1x05-P0.5mm -> Connector_PinHeader_2.54mm:PinHeader_1x05_P2.54mm_Vertical
- R1, R11, R13, R15, R17, R19, R21, R23, TPA15, TPA8, TPB1, TPB10, TPB12, TPB2, TPB3, TPB4, TPB5, TPB8, TPB9, TPC0, TPC1, TPC10, TPC11, TPC13, TPC14, TPC15, TPC2, TPC3, TPC6, TPC7, TPC8, TPC9, TPD2: moved to B.Cu
- SW2: footprint Button_Switch_SMD:SW_SP3T_PCM13 -> Button_Switch_SMD:SW_Push_SPST_NO_Alps_SKRK
- moved J1 121.7 mm to (55.3, 134.4), turned to 180 degrees
- moved J2 103.2 mm to (52.8, 38.0), turned to 0 degrees
- moved TPA8 12.3 mm to (55.6, 72.5)
- moved TPB12 12.3 mm to (61.7, 72.5)
- moved TPB4 12.3 mm to (58.6, 72.5)
- moved TPC11 12.3 mm to (67.8, 72.5)
- moved TPC6 12.3 mm to (64.8, 72.5)
- moved TPB10 12.1 mm to (58.6, 60.2)
- moved TPB3 12.1 mm to (55.6, 60.2)
- moved TPC10 12.1 mm to (64.8, 60.2)
- moved TPC3 12.1 mm to (61.7, 60.2)
- moved TPD2 12.1 mm to (67.8, 60.2)
- moved TPA15 6.20 mm to (55.6, 69.4)
- moved TPB5 6.20 mm to (58.6, 69.4)
- moved TPC0 6.20 mm to (61.7, 69.4)
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Connections:
- J2 pad 1: (no net) -> GND
- J2 pad 2: (no net) -> /TX
- J2 pad 3: (no net) -> /RX
- J2 pad 4: (no net) -> /SWDIO
- J2 pad 5: (no net) -> /SWCLK

Commit message: hw: finish layout
Parts:
- added kibuzzard-682DE080: G***, kibuzzard-682DE080, F.Cu at (55.5, 140.0)
- added kibuzzard-682DE088: G***, kibuzzard-682DE088, F.Cu at (55.5, 144.6)
- added kibuzzard-682DECE7: G***, kibuzzard-682DECE7, F.Cu at (55.5, 147.2)
- added kibuzzard-682DFB76: G***, kibuzzard-682DFB76, F.Cu at (55.5, 149.8)
- added kibuzzard-682DFB84: G***, kibuzzard-682DFB84, F.Cu at (55.5, 152.4)
- added kibuzzard-682DFB98: G***, kibuzzard-682DFB98, F.Cu at (55.5, 155.0)
- moved R14 151.8 mm to (189.1, 38.0)
- moved R12 134.2 mm to (164.9, 38.0)
- moved R9 119.1 mm to (140.0, 37.5)
- moved J2 116.9 mm to (50.2, 154.9), turned to 180 degrees
- moved R7 116.4 mm to (57.0, 35.0), turned to 180 degrees
- moved R3 111.2 mm to (115.6, 36.5)
- moved R8 105.9 mm to (64.0, 35.0)
- moved R22 104.6 mm to (189.4, 149.0)
- moved C5 102.8 mm to (105.5, 45.9), turned to 90 degrees
- moved C4 99.3 mm to (90.0, 46.1), turned to 90 degrees
- moved C3 98.3 mm to (75.0, 45.9), turned to 90 degrees
- moved C28 91.9 mm to (72.8, 31.5), turned to -90 degrees
- moved C13 88.1 mm to (86.8, 32.0), turned to 90 degrees
- moved SW4 85.1 mm to (83.8, 46.2)
- moved U5 83.2 mm to (80.0, 31.5), turned to -90 degrees
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Connections:
- net /USB_DM renamed /USB_D-
- net /USB_DP renamed /USB_D+
- U1 pad 14: /ADC_CH0 -> /ADC_CH5
- U1 pad 15: /ADC_CH1 -> /ADC_CH6
- U1 pad 16: /ADC_CH2 -> /ADC_CH7
- U1 pad 17: /ADC_CH3 -> /ADC_CH4
- U1 pad 20: /ADC_CH4 -> /ADC_CH3
- U1 pad 21: /ADC_CH5 -> /ADC_CH2
- U1 pad 22: /ADC_CH6 -> /ADC_CH1
- U1 pad 23: /ADC_CH7 -> /ADC_CH0
- Y1 pad 2: /OSC_IN -> GND
- Y1 pad 3: (no net) -> /OSC_IN
- Y1 pad 4: (no net) -> GND
Routing:
- net /USB_D-: track 0.00 -> 46.3 mm
- net /USB_D+: track 0.00 -> 46.1 mm
- net Net-(U1-PA12): track 0.00 -> 27.4 mm
- net 5V: track 0.00 -> 26.2 mm
- net Net-(U1-PA11): track 0.00 -> 25.6 mm
- net GND: track 0.00 -> 15.0 mm
- net 3.3V: track 0.00 -> 13.7 mm
- net VDDA: track 0.00 -> 9.15 mm
- net Net-(J4-CC1): track 0.00 -> 5.32 mm
- net Net-(J4-CC2): track 0.00 -> 4.60 mm
- added copper zone on F.Cu, net 3.3V
- added copper zone on F.Cu, net 5V
- added copper zone on B.Cu, net GND
Other:
- board outline added: 156.1 x 134.5 mm

Commit message: hw: start routing
Parts:
- removed kibuzzard-682DE088: G***, kibuzzard-682DE088
- removed kibuzzard-682DECE7: G***, kibuzzard-682DECE7
- removed kibuzzard-682DFB76: G***, kibuzzard-682DFB76
- removed kibuzzard-682DFB84: G***, kibuzzard-682DFB84
- removed kibuzzard-682DFB98: G***, kibuzzard-682DFB98
- moved J5 152.7 mm to (201.6, 155.9), turned to 180 degrees
- moved kibuzzard-682DE080 146.5 mm to (201.6, 150.5), turned to 90 degrees
- moved J2 78.8 mm to (50.0, 76.0), turned to 0 degrees
- moved C3 8.78 mm to (68.5, 51.8), turned to 0 degrees
- moved C7 0.58 mm to (94.0, 88.3)
- turned R2 to 135 degrees
Connections:
- D1 pad 4: /LED_IN -> /LED_5050x8/LED_IN
- D10 pad 4: /LED_2020_Trimmer/LED_IN -> /LED_IN
- D20 pad 2: /LED_play_pause_mode/LED_OUT -> /LED_5050x8/LED_IN
- D8 pad 2: /LED_2020_Trimmer/LED_IN -> /LED_5050x8/LED_OUT
- J5 pad 1: /LED_play_pause_mode/LED_OUT -> /LED_5050x8/LED_OUT
Routing:
- net 5V: track 26.2 -> 585.2 mm, vias 0 -> 12
- net 3.3V: track 13.7 -> 311.6 mm, vias 0 -> 4
- net Net-(D4-DOUT): track 0.00 -> 240.1 mm, vias 0 -> 2
- net /ADC_CH7: track 0.00 -> 157.7 mm, vias 0 -> 5
- net /ADC_CH3: track 0.00 -> 144.5 mm, vias 0 -> 1
- net /ADC_CH6: track 0.00 -> 132.2 mm, vias 0 -> 3
- net /ADC_CH2: track 0.00 -> 122.0 mm, vias 0 -> 5
- net GND: track 15.0 -> 128.8 mm, vias 0 -> 54
- net /SCL: track 0.00 -> 110.5 mm, vias 0 -> 1
- net /SDA: track 0.00 -> 110.1 mm, vias 0 -> 1
- net /ADC_CH5: track 0.00 -> 107.7 mm, vias 0 -> 3
- net /ADC_CH1: track 0.00 -> 99.3 mm, vias 0 -> 3
- net /ADC_CH4: track 0.00 -> 81.7 mm, vias 0 -> 3
- net /ADC_CH0: track 0.00 -> 75.6 mm, vias 0 -> 3
- net Net-(D5-DOUT): track 0.00 -> 75.5 mm, vias 0 -> 7
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
Commit message: hw: finish routing
Parts:
- moved TPB10 15.1 mm to (83.4, 92.2)
- moved TPC14 9.96 mm to (91.5, 116.0)
- moved TPB5 7.02 mm to (67.5, 112.5)
Routing:
- net Net-(U1-PB9): track 0.00 -> 30.9 mm, vias 0 -> 1
- net Net-(U1-PB8): track 0.00 -> 28.9 mm, vias 0 -> 1
- net Net-(U1-PB4): track 0.00 -> 23.7 mm, vias 0 -> 1
- net GND: track 128.8 -> 152.3 mm, vias 54 -> 58
- net Net-(U1-PB3): track 0.00 -> 23.2 mm, vias 0 -> 3
- net Net-(U1-PC2): track 0.00 -> 22.2 mm, vias 0 -> 1
- net Net-(U1-PC15): track 0.00 -> 20.9 mm, vias 0 -> 1
- net Net-(U1-PB5): track 0.00 -> 20.6 mm, vias 0 -> 3
- net Net-(U1-PC14): track 0.00 -> 18.8 mm, vias 0 -> 1
- net Net-(U1-PC13): track 0.00 -> 18.8 mm, vias 0 -> 1
- net Net-(U1-PB1): track 0.00 -> 17.2 mm, vias 0 -> 2
- net Net-(U1-PC3): track 0.00 -> 17.0 mm, vias 0 -> 1
- net Net-(U1-PC1): track 0.00 -> 15.0 mm, vias 0 -> 1
- net Net-(U1-PB2): track 0.00 -> 14.2 mm, vias 0 -> 3
- net Net-(U1-PC0): track 0.00 -> 9.57 mm, vias 0 -> 1
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
Commit message: hw: add GND plane
Routing:
- net GND: track 152.3 -> 127.7 mm, vias 58 -> 42
- added copper zone on F.Cu, net GND

Commit message: hw: added esd protection and caps
Parts:
- added C34: DNF, Capacitor_SMD:C_0402_1005Metric_Pad0.74x0.62mm_HandSolder, F.Cu at (115.6, 30.6)
- added C35: DNF, Capacitor_SMD:C_0402_1005Metric_Pad0.74x0.62mm_HandSolder, F.Cu at (139.9, 30.6)
- added C36: DNF, Capacitor_SMD:C_0402_1005Metric_Pad0.74x0.62mm_HandSolder, F.Cu at (164.4, 30.6)
- added C37: DNF, Capacitor_SMD:C_0402_1005Metric_Pad0.74x0.62mm_HandSolder, F.Cu at (189.0, 30.6)
- added C38: DNF, Capacitor_SMD:C_0402_1005Metric_Pad0.74x0.62mm_HandSolder, F.Cu at (115.3, 155.8)
- added C39: DNF, Capacitor_SMD:C_0402_1005Metric_Pad0.74x0.62mm_HandSolder, F.Cu at (140.0, 155.8)
- added C40: DNF, Capacitor_SMD:C_0402_1005Metric_Pad0.74x0.62mm_HandSolder, F.Cu at (164.4, 155.8)
- added C41: DNF, Capacitor_SMD:C_0402_1005Metric_Pad0.74x0.62mm_HandSolder, F.Cu at (189.0, 155.8)
- added C42: DNF, Capacitor_SMD:C_0402_1005Metric_Pad0.74x0.62mm_HandSolder, F.Cu at (86.4, 79.0)
- added U2: USBLC6-2SC6, Package_TO_SOT_SMD:SOT-23-6, F.Cu at (59.8, 39.2)
- added kibuzzard-682F341C: G***, kibuzzard-682F341C, F.Cu at (54.2, 76.0)
- added kibuzzard-682F3431: G***, kibuzzard-682F3431, F.Cu at (54.2, 78.5)
- added kibuzzard-682F3436: G***, kibuzzard-682F3436, F.Cu at (54.2, 81.2)
- added kibuzzard-682F343C: G***, kibuzzard-682F343C, F.Cu at (54.2, 83.8)
- added kibuzzard-682F3442: G***, kibuzzard-682F3442, F.Cu at (54.2, 86.2)
- added kibuzzard-682F3456: G***, kibuzzard-682F3456, F.Cu at (68.8, 25.5)
- moved J5 0.10 mm to (201.6, 156.0), turned to 0 degrees
Connections:
- J4 pad A6: /USB_D+ -> Net-(J4-D+-PadA6)
- J4 pad A7: /USB_D- -> Net-(J4-D--PadA7)
- J4 pad B6: /USB_D+ -> Net-(J4-D+-PadA6)
- J4 pad B7: /USB_D- -> Net-(J4-D--PadA7)
- J5 pad 1: /LED_5050x8/LED_OUT -> (no net)
Routing:
- net /USB_D-: track 46.3 -> 33.7 mm
- net /USB_D+: track 46.1 -> 34.4 mm
- net Net-(J4-D--PadA7): track 0.00 -> 10.3 mm
- net Net-(J4-D+-PadA6): track 0.00 -> 10.2 mm
- net GND: track 127.7 -> 136.3 mm, vias 42 -> 1342
- net 5V: track 592.4 -> 600.0 mm
- net /ADC_CH8: track 18.3 -> 23.0 mm
- net /ADC_CH0: track 75.6 -> 77.1 mm, vias 3 -> 4
- net /ADC_CH3: track 144.5 -> 145.9 mm, vias 1 -> 2
- net /ADC_CH1: track 99.3 -> 100.7 mm, vias 3 -> 4
- net /ADC_CH6: track 132.2 -> 133.6 mm, vias 3 -> 4
- net /ADC_CH7: track 157.7 -> 159.0 mm, vias 5 -> 6
- net /ADC_CH2: track 122.0 -> 123.3 mm, vias 5 -> 6
- net /ADC_CH4: track 81.7 -> 82.9 mm, vias 3 -> 4
- net /ADC_CH5: track 107.7 -> 108.8 mm, vias 3 -> 4

Commit message: hw: silkscreen
Routing:
- net /SDA: track 118.4 -> 117.6 mm
Changed lines of the file:
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@@
 				(font
 					(size 0.001 0.001)
+					(thickness 0.15)
 				)
 			)
@@
 				(font
 					(size 0.001 0.001)
+					(thickness 0.15)
 				)
 			)
@@
 		(tags "capacitor handsolder")
 		(property "Reference" "C13"
-			(at 0 -1.68 90)
+			(at -0.166666 -1.987086 90)
 			(layer "F.SilkS")
 			(effects
@@
 				(font
 					(size 0.001 0.001)
+					(thickness 0.15)
 				)
 			)
@@
 				(font
 					(size 0.001 0.001)
+					(thickness 0.15)
 				)
 			)
@@
 		(tags "LQFP QFP")
 		(property "Reference" "U1"
-			(at 0 -0.5 315)
+			(at 1 -1.1 315)
 			(layer "F.SilkS")
 			(effects
@@
 		(descr "SMD3225/4, Crystal, 3.2x2.5mm package, SMD, generated with kicad-footprint-generator make_crystal.py, http://www.txccrystal.com/images/pdf/7m-accuracy.pdf")
 		(property "Reference" "Y1"
-			(at 2.828427 0 135)
+			(at 2.828427 -0.565685 135)
 			(layer "F.SilkS")
 			(effects
@@
 		(tags "LED RGB NeoPixel Nano PLCC-4 2020")
 		(property "Reference" "D14"
-			(at 0 -2 0)
+			(at 0 2.18 0)
 			(layer "F.SilkS")
 			(effects
@@
 				(font
 					(size 0.001 0.001)
+					(thickness 0.15)
 				)
 			)
@@
 				(font
 					(size 0.001 0.001)
+					(thickness 0.15)
 				)
 			)
@@
 		(tags "capacitor handsolder")
 		(property "Reference" "C24"
-			(at -2.42 -0.1 180)
+			(at -1.92 0.1 180)
 			(layer "F.SilkS")
 			(effects
@@
 		(tags "capacitor handsolder")
 		(property "Reference" "C25"
-			(at 0 -1.16 0)
+			(at -2.8 0.001796 0)
 			(layer "F.SilkS")
 			(effects
@@
 		(tags "resistor handsolder")
 		(property "Reference" "R2"
-			(at 0 1.414214 135)
+			(at -2.12132 0 135)
 			(layer "F.SilkS")
 			(effects
@@
 		(tags "capacitor handsolder")
 		(property "Reference" "C1"
-			(at 0 -1.16 45)
+			(at -0.001814 -1.697056 45)
 			(layer "F.SilkS")
 			(effects
@@
 		(tags "CMS SOT")
 		(property "Reference" "U5"
-			(at 0 -4.5 90)
+			(at -5.3 0 180)
 			(layer "F.SilkS")
 			(effects
@@
 		(tags "LED RGB NeoPixel Nano PLCC-4 2020")
 		(property "Reference" "D15"
-			(at 0 -2 0)
+			(at 0.15 2.18 0)
 			(layer "F.SilkS")
 			(effects
@@
 				(font
 					(size 0.001 0.001)
+					(thickness 0.15)
 				)
 			)
@@
 				(font
 					(size 0.001 0.001)
+					(thickness 0.15)
 				)
 			)
@@
 				(font
 					(size 0.001 0.001)
+					(thickness 0.15)
 				)
 			)
@@
 				(font
 					(size 0.001 0.001)
+					(thickness 0.15)
 				)
 			)
@@
 				(font
 					(size 0.001 0.001)
+					(thickness 0.15)
 				)
 			)
@@
 				(font
 					(size 0.001 0.001)
+					(thickness 0.15)
 				)
 			)
@@
 		(tags "SMD SMT button")
 		(property "Reference" "SW2"
-			(at 1.59099 -1.59099 0)
+			(at 1.767767 -1.767767 0)
 			(layer "F.SilkS")
 			(effects
@@
 		(tags "LED RGB NeoPixel Nano PLCC-4 2020")
 		(property "Reference" "D13"
-			(at 0 -2 0)
+			(at 0 2.08 0)
 			(layer "F.SilkS")
 			(effects
@@
 	)
 	(segment
+		(start 77 78.474341)
+		(end 85.361179 86.83552)
+		(width 0.25)
+		(layer "F.Cu")
+		(net 7)
+	)
+	(segment
 		(start 165.605 36.7)
 		(end 187.2 36.7)
@@
 	)
 	(segment
-		(start 77 78.474341)
-		(end 85.361179 86.83552)
-		(width 0.25)
-		(layer "F.Cu")
-		(net 7)
-	)
-	(segment
 		(start 141.9 150.4)
 		(end 139.5 148)
@@
 	)
 	(segment
-		(start 88.425 91.810917)
-		(end 88.335917 91.9)
-		(width 0.2)
-		(layer "B.Cu")
-		(net 40)
-	)
-	(segment
 		(start 90.302 89.933916)
 		(end 90.302 78.848056)
@@
 	)
 	(segment
-		(start 99.299 69.851057)
-		(end 99.775028 69.375028)
-		(width 0.2)
-		(layer "B.Cu")
-		(net 40)
-	)
-	(segment
-		(start 88.317958 91.917958)
-		(end 88.335917 91.9)
-		(width 0.2)
-		(layer "B.Cu")
-		(net 40)
-	)
-	(segment
 		(start 131.28 54.3)
 		(end 155.58 30)
@@
 	)
 	(segment
+		(start 154.4 49.9)
+		(end 166.6 37.7)
+		(width 0.25)
+		(layer "F.Cu")
+		(net 44)
+	)
+	(segment
+		(start 166.6 37.7)
+		(end 166.6 37.5)
+		(width 0.25)
+		(layer "F.Cu")
+		(net 44)
+	)
+	(segment
 		(start 115.9 60.4)
 		(end 115.9 53.5)
@@
 	)
 	(segment
-		(start 154.4 49.9)
-		(end 167 37.3)
-		(width 0.25)
-		(layer "F.Cu")
-		(net 44)
-	)
-	(segment
 		(start 166 37.5)
 		(end 165.5 38)
@@
 		)
 	)
-	(group ""
-		(members "33d18e38-ca5c-4d63-b5bc-11531a0dda68" "39344536-da8a-4050-9df9-901fb2a0dfae"
-			"53649017-9595-4e18-841b-06db2e8aa72e" "5755208f-91da-4375-8e69-e36a95b00dfa"
-			"57fad9b6-05ac-4040-b06c-0101c93212cc" "76016e02-b90f-46d4-8354-b101c411bc2c"
-			"7ad7074b-35c8-4d33-a003-47f45cedb617" "97d6ff5d-25c2-41d7-9e1e-f76bbe7a10e7"
-			"a37900c9-9cf4-4e3b-8c86-1052c81867a8" "a4925f19-02c5-4076-8149-9773e55144b7"
-			"b40748ae-1e16-42ad-9a3d-b92caa719558" "ba126b38-ea71-4a72-92f7-99c49c820e93"
-			"cca2cb6f-775d-4037-bd5e-0a5bbbb62509" "d5531db1-bd7e-48eb-96ed-0855ee9d4db9"
-			"ddae3e7e-eeaa-4755-9be1-12f39d00e336" "f42c72af-8e97-4868-9eef-50836a71eab8"
-			"f84fac71-1e6a-4740-883c-e8db57fb03fa"
-		)
-	)

Commit message: hw: fix drc errors
Connections:
- J5 pad 1: (no net) -> /LED_5050x8/LED_OUT
Routing:
- net 5V: track 600.0 -> 591.4 mm
- net Net-(U1-PB1): track 17.2 -> 17.1 mm, vias 2 -> 1
Changed lines of the file:
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@@
 			)
 		)
+		(property ki_fp_filters "Connector*:*_1x??_*")
+		(sheetname "/")
+		(sheetfile "gigasound-hw.kicad_sch")
 		(attr through_hole)
 		(fp_line
@@
 			(layers "*.Cu" "*.Mask")
 			(remove_unused_layers no)
+			(net 31 "/LED_5050x8/LED_OUT")
 			(pinfunction "Pin_1")
 			(pintype "passive")
@@
 		)
 		(embedded_fonts no)
-		(embedded_files
-			(file
-				(name "Switch JoyCon joystick v2.step")
-				(type model)
-				(checksum "DE4A15B77536FDE44B24A35898A78697")
-			)
-		)
-		(model "kicad-embed://Switch JoyCon joystick v2.step"
-			(offset
-				(xyz 35 -120.5 0)
-			)
-			(scale
-				(xyz 1 1 1)
-			)
-			(rotate
-				(xyz -0 90 -0)
-			)
-		)
 	)
 	(footprint "LED_SMD:LED_WS2812B_PLCC4_5.0x5.0mm_P3.2mm"
@@
 	)
 	(segment
+		(start 127.9 62)
+		(end 127.9 142)
+		(width 1)
+		(layer "F.Cu")
+		(net 11)
+	)
+	(segment
+		(start 127.9 52.1)
+		(end 127.9 57.1)
+		(width 1)
+		(layer "F.Cu")
+		(net 11)
+	)
+	(segment
 		(start 57.49 30.62)
 		(end 57.49 29.824587)
@@
 	)
 	(segment
-		(start 128 62.1)
-		(end 128 142)
-		(width 1)
-		(layer "F.Cu")
-		(net 11)
-	)
-	(segment
 		(start 161.866666 53.633334)
 		(end 163.5 52)
@@
 	)
 	(segment
-		(start 128 142)
-		(end 128.5 142)
-		(width 1)
-		(layer "F.Cu")
-		(net 11)
-	)
-	(segment
 		(start 161.96 76.193334)
 		(end 161.866666 76.1)
@@
 	)
 	(segment
-		(start 127.9 62)
-		(end 128 62.1)
-		(width 1)
-		(layer "F.Cu")
-		(net 11)
-	)
-	(segment
 		(start 72.5 60.3)
 		(end 73.1 60.9)
@@
 	)
 	(segment
-		(start 127.8 52)
-		(end 127.8 57)
-		(width 1)
-		(layer "F.Cu")
-		(net 11)
-	)
-	(segment
 		(start 60.037501 39.4)
 		(end 61.475 39.4)
@@
 	)
 	(segment
-		(start 98.07 39.95)
-		(end 97.52 39.95)
-		(width 0.2)
+		(start 127.8 52)
+		(end 127.9 52.1)
+		(width 1)
 		(layer "F.Cu")
 		(net 11)
 	)
 	(segment
-		(start 189.3 142)
-		(end 197.4 142)
-		(width 1)
+		(start 98.07 39.95)
+		(end 97.52 39.95)
+		(width 0.2)
 		(layer "F.Cu")
 		(net 11)
@@
 	)
 	(segment
-		(start 197.4 142)
-		(end 197.7 142.3)
-		(width 1)
-		(layer "F.Cu")
-		(net 11)
-	)
-	(segment
 		(start 72.75 30.4625)
 		(end 72.75 28.6)
@@
 	)
 	(segment
-		(start 112.865 53.3)
-		(end 112.865 53.135)
-		(width 0.3)
-		(layer "F.Cu")
-		(net 11)
-	)
-	(segment
 		(start 112.865 52.686)
 		(end 113.551 52)
@@
 	)
 	(segment
-		(start 127.8 57)
-		(end 127.9 57.1)
-		(width 1)
-		(layer "F.Cu")
-		(net 11)
-	)
-	(segment
 		(start 164.3 52)
 		(end 187.2 52)
@@
 		(net 11)
 	)
+	(segment
+		(start 127.9 142)
+		(end 128.5 142)
+		(width 1)
+		(layer "F.Cu")
+		(net 11)
+	)
 	(via
 		(at 84.9 61.9)
@@
 	)
 	(segment
-		(start 122.7 143.9)
-		(end 122.8 143.8)
-		(width 0.25)
-		(layer "F.Cu")
-		(net 16)
-	)
-	(segment
 		(start 202.3 141.7)
 		(end 200.1 143.9)
@@
 	)
 	(segment
-		(start 116.2 137.2)
-		(end 116.2 137)
-		(width 0.25)
-		(layer "F.Cu")
-		(net 16)
-	)
-	(segment
 		(start 119.1 140.5)
 		(end 116.2 137.6)
@@
 	)
 	(segment
-		(start 88.5 92.454328)
-		(end 87.498419 92.454328)
+		(start 87.498419 92.454328)
+		(end 86 90.955909)
 		(width 0.2)
 		(layer "F.Cu")
@@
 	)
 	(segment
-		(start 87.498419 92.454328)
-		(end 86 90.955909)
+		(start 88.565059 92.519387)
+		(end 88.5 92.454328)
 		(width 0.2)
 		(layer "F.Cu")
@@
 	)
 	(segment
-		(start 86 90.955909)
-		(end 86 89.5)
+		(start 86 89.7)
+		(end 87.096713 88.603287)
 		(width 0.2)
 		(layer "F.Cu")
@@
 	)
 	(segment
-		(start 88.565059 92.519387)
-		(end 88.5 92.454328)
+		(start 88.5 92.454328)
+		(end 87.498419 92.454328)
 		(width 0.2)
 		(layer "F.Cu")
@@
 	)
 	(segment
-		(start 86.232233 89.5)
-		(end 86 89.5)
+		(start 86 90.955909)
+		(end 86 89.7)
 		(width 0.2)
 		(layer "F.Cu")
@@
 	)
 	(segment
-		(start 87.128946 88.603287)
-		(end 86.232233 89.5)
+		(start 87.096713 88.603287)
+		(end 87.128946 88.603287)
 		(width 0.2)
 		(layer "F.Cu")
 		(net 55)
 	)
-	(via
-		(at 86 89.5)
-		(size 0.6)
-		(drill 0.3)
-		(layers "F.Cu" "B.Cu")
-		(net 55)
-	)
