File: gigasound-hw/gigasound-hw.kicad_pcb (KiCad board)
At the start: 2 copper layers, 156.1 x 134.5 mm, 143 parts, among them J1 Conn_01x05_Socket_FPC_Joycon, J2 Conn_01x05_Socket_UART, J4 USB_C_Receptacle_USB2.0_16P, J5 PIN_LED_OUT, J6 Conn_01x04_Socket_OLED, SW1 PLAY, SW2 Reset, SW4 STOP, SW5 MODE, U1 STM32F401RETx, U2 USBLC6-2SC6, U5 AMS1117-3.3, Y1 12MHz

Commit message: hw: new pcb revision candidate
Parts:
- turned C11 to 45 degrees
Other:
- board text added: "Rev. 1.1-rc0"
- board text removed: "Rev. 1.0"
Changed lines of the file:
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@@
 	(footprint "Capacitor_SMD:C_0402_1005Metric_Pad0.74x0.62mm_HandSolder"
 		(layer "F.Cu")
-		(at 95.694177 97.305823 -135)
+		(at 95.694177 97.305823 45)
 		(descr "Capacitor SMD 0402 (1005 Metric), square (rectangular) end terminal, IPC-7351 nominal with elongated pad for handsoldering. (Body size source: IPC-SM-782 page 76, https://www.pcb-3d.com/wordpress/wp-content/uploads/ipc-sm-782a_amendment_1_and_2.pdf), generated with kicad-footprint-generator")
 		(tags "capacitor handsolder")
@@
 		(attr smd)
 		(fp_line
-			(start -0.115835 0.36)
-			(end 0.115835 0.36)
+			(start -0.115835 -0.36)
+			(end 0.115835 -0.36)
 			(stroke
 				(width 0.12)
@@
 		)
 		(fp_line
-			(start -0.115835 -0.36)
-			(end 0.115835 -0.36)
+			(start -0.115835 0.36)
+			(end 0.115835 0.36)
 			(stroke
 				(width 0.12)
@@
 		)
 		(fp_line
-			(start 1.09 0.460001)
-			(end -1.09 0.460001)
+			(start -1.09 -0.460001)
+			(end 1.09 -0.460001)
 			(stroke
 				(width 0.05)
@@
 		)
 		(fp_line
-			(start 1.09 -0.460001)
-			(end 1.09 0.460001)
+			(start -1.09 0.460001)
+			(end -1.09 -0.460001)
 			(stroke
 				(width 0.05)
@@
 		)
 		(fp_line
-			(start -1.09 0.460001)
-			(end -1.09 -0.460001)
+			(start 1.09 -0.460001)
+			(end 1.09 0.460001)
 			(stroke
 				(width 0.05)
@@
 		)
 		(fp_line
-			(start -1.09 -0.460001)
-			(end 1.09 -0.460001)
+			(start 1.09 0.460001)
+			(end -1.09 0.460001)
 			(stroke
 				(width 0.05)
@@
 		)
 		(fp_line
-			(start 0.5 0.25)
-			(end -0.5 0.25)
+			(start -0.5 -0.25)
+			(end 0.5 -0.25)
 			(stroke
 				(width 0.1)
@@
 		)
 		(fp_line
-			(start 0.5 -0.25)
-			(end 0.5 0.25)
+			(start -0.5 0.25)
+			(end -0.5 -0.25)
 			(stroke
 				(width 0.1)
@@
 		)
 		(fp_line
-			(start -0.5 0.25)
-			(end -0.5 -0.25)
+			(start 0.5 -0.25)
+			(end 0.5 0.25)
 			(stroke
 				(width 0.1)
@@
 		)
 		(fp_line
-			(start -0.5 -0.25)
-			(end 0.5 -0.25)
+			(start 0.5 0.25)
+			(end -0.5 0.25)
 			(stroke
 				(width 0.1)
@@
 		)
 		(pad "1" smd roundrect
-			(at -0.5675 0 225)
+			(at -0.5675 0 45)
 			(size 0.735 0.62)
 			(layers "F.Cu" "F.Mask" "F.Paste")
@@
 		)
 		(pad "2" smd roundrect
-			(at 0.5675 0 225)
+			(at 0.5675 0 45)
 			(size 0.735 0.62)
 			(layers "F.Cu" "F.Mask" "F.Paste")
@@
 		(layer "Edge.Cuts")
 	)
-	(gr_text "Rev. 1.0"
+	(gr_text "Rev. 1.1-rc0"
 		(at 173.2 143.4 0)
 		(layer "B.SilkS")
@@
 	)
 	(segment
-		(start 93.60586 96.894764)
-		(end 95.087101 98.376005)
-		(width 0.2)
-		(layer "F.Cu")
-		(net 2)
-	)
-	(segment
 		(start 87.875 30.925)
 		(end 89 29.8)
@@
 	)
 	(segment
-		(start 95.417369 98.376005)
-		(end 96.09546 97.697914)
-		(width 0.2)
-		(layer "F.Cu")
-		(net 2)
-	)
-	(segment
 		(start 69.035 51.8)
 		(end 70 51.8)
@@
 	)
 	(segment
-		(start 95.087101 98.376005)
-		(end 95.417369 98.376005)
-		(width 0.2)
-		(layer "F.Cu")
-		(net 2)
-	)
-	(segment
 		(start 93.315 69.87)
 		(end 94.9825 69.87)
@@
 	)
 	(segment
+		(start 96.09546 96.90454)
+		(end 96.09546 97.697914)
+		(width 0.2)
+		(layer "F.Cu")
+		(net 2)
+	)
+	(segment
 		(start 90 45.5)
 		(end 90.9 45.5)
@@
 	)
 	(segment
-		(start 96.09546 97.697914)
-		(end 96.09546 96.90454)
-		(width 0.2)
-		(layer "F.Cu")
-		(net 2)
-	)
-	(segment
 		(start 56.6 98.5)
 		(end 56.6 94.375647)
@@
 	)
 	(segment
-		(start 89.869636 96.894764)
-		(end 93.60586 96.894764)
-		(width 0.2)
+		(start 94.9825 69.87)
+		(end 95 69.8875)
+		(width 0.25)
 		(layer "F.Cu")
 		(net 2)
 	)
 	(segment
-		(start 94.9825 69.87)
-		(end 95 69.8875)
-		(width 0.25)
+		(start 95.087101 98.376005)
+		(end 93.60586 96.894764)
+		(width 0.2)
 		(layer "F.Cu")
 		(net 2)
@@
 	)
 	(segment
+		(start 95.417369 98.376005)
+		(end 95.087101 98.376005)
+		(width 0.2)
+		(layer "F.Cu")
+		(net 2)
+	)
+	(segment
 		(start 63.09 30.62)
 		(end 63.09 31.06)
@@
 	)
 	(segment
-		(start 89.250266 96.275394)
-		(end 89.869636 96.894764)
-		(width 0.2)
+		(start 65.35 44.35)
+		(end 63.65 44.35)
+		(width 0.25)
 		(layer "F.Cu")
 		(net 2)
 	)
 	(segment
-		(start 65.35 44.35)
-		(end 63.65 44.35)
-		(width 0.25)
+		(start 93.60586 96.894764)
+		(end 89.869636 96.894764)
+		(width 0.2)
 		(layer "F.Cu")
 		(net 2)
@@
 		(layer "F.Cu")
 		(net 2)
+	)
+	(segment
+		(start 89.869636 96.894764)
+		(end 89.250266 96.275394)
+		(width 0.2)
+		(layer "F.Cu")
+		(net 2)
+	)
+	(segment
+		(start 96.09546 97.697914)
+		(end 95.417369 98.376005)
+		(width 0.2)
+		(layer "F.Cu")
+		(net 2)
