File: gigasound-hw/gigasound-hw.kicad_sch (KiCad schematic)
At the start: 75 parts, among them J1 Conn_01x04_Socket, J2 Conn_01x05_Socket, J3 Conn_01x05_Socket, J4 USB_C_Receptacle_USB2.0_16P, J5 PIN_LED_OUT, SW1 PLAY, SW2 100nF, SW4 STOP, SW5 MODE, U1 STM32F401RETx, U5 AMS1117-3.3, Y1 8MHz

Commit message: add footprint
Parts:
- added R24, R25: 0, Resistor_SMD:R_0402_1005Metric_Pad0.72x0.64mm_HandSolder, symbol Device:R
- C1, C2: value C -> 7.5pF; footprint (none) -> Capacitor_SMD:C_0402_1005Metric_Pad0.74x0.62mm_HandSolder
- C10, C11, C3, C4, C5, C6, C7, C8, C9: footprint (none) -> Capacitor_SMD:C_0402_1005Metric_Pad0.74x0.62mm_HandSolder
- C12: footprint (none) -> Capacitor_SMD:C_0805_2012Metric_Pad1.18x1.45mm_HandSolder
- C13, C28: footprint Capacitor_SMD:C_0402_1005Metric_Pad0.74x0.62mm_HandSolder -> Capacitor_SMD:C_0805_2012Metric_Pad1.18x1.45mm_HandSolder
- J3: footprint (none) -> Connector_PinHeader_2.54mm:PinHeader_1x04_P2.54mm_Vertical
- L1: footprint (none) -> Inductor_SMD:L_0201_0603Metric_Pad0.64x0.40mm_HandSolder
- R12, R14, R16, R18, R20, R22, R3, R4, R5, R6, R9: footprint (none) -> Resistor_SMD:R_0402_1005Metric_Pad0.72x0.64mm_HandSolder
- R2: value R -> 1K; footprint (none) -> Resistor_SMD:R_0402_1005Metric_Pad0.72x0.64mm_HandSolder
- RV1: value R_Potentiometer_Trim -> 100K; footprint Potentiometer_THT:Potentiometer_Piher_PT-10-V10_Vertical -> Potentiometer_THT:Potentiometer_Alps_RK09K_Single_Vertical
- SW2: value 100nF -> ~
- Y1: value 8MHz -> 12MHz; footprint Crystal:Crystal_SMD_SeikoEpson_MA505-2Pin_12.7x5.1mm_HandSoldering -> Crystal:Crystal_SMD_3225-4Pin_3.2x2.5mm
Connections:
- net USB_DM: now also R25.2; no longer U1.44 (PA11)
- net USB_DP: now also R24.2; no longer U1.45 (PA12)
- new net: R24.1, U1.45 (PA12)
- new net: R25.1, U1.44 (PA11)
Other:
- note added: "ABM8-272-T3"
- note removed: "scegliere C e R in base al cristallo definitivo"

Commit message: hw: footprints
Parts:
- J2: footprint (none) -> gigalibrary:Joycon-FPC-1x05-P0.5mm
- R1, R11, R13, R15, R17, R19, R21, R23: footprint (none) -> gigalibrary:FSR402
- SW1, SW4, SW5: footprint (none) -> Button_Switch_SMD:SW_SPST_TL3342
- SW2: value ~ -> Reset; footprint (none) -> Button_Switch_SMD:SW_SP3T_PCM13
Changed lines of the file:
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@@
 			)
 		)
-		(property "Footprint" ""
+		(property "Footprint" "gigalibrary:FSR402"
 			(at 243.332 58.42 90)
 			(effects
@@
 			)
 		)
-		(property "Footprint" ""
+		(property "Footprint" "gigalibrary:Joycon-FPC-1x05-P0.5mm"
 			(at 121.92 143.51 0)
 			(effects
@@
 			)
 		)
-		(property "Footprint" ""
+		(property "Footprint" "gigalibrary:FSR402"
 			(at 205.232 58.42 90)
 			(effects
@@
 			)
 		)
-		(property "Footprint" ""
+		(property "Footprint" "Button_Switch_SMD:SW_SPST_TL3342"
 			(at 176.53 83.82 0)
 			(effects
@@
 			)
 		)
-		(property "Footprint" ""
+		(property "Footprint" "gigalibrary:FSR402"
 			(at 263.652 58.42 90)
 			(effects
@@
 			)
 		)
-		(property "Footprint" ""
+		(property "Footprint" "gigalibrary:FSR402"
 			(at 224.282 58.42 90)
 			(effects
@@
 			)
 		)
-		(property "Footprint" ""
+		(property "Footprint" "gigalibrary:FSR402"
 			(at 167.132 58.42 90)
 			(effects
@@
 			)
 		)
-		(property "Footprint" ""
+		(property "Footprint" "gigalibrary:FSR402"
 			(at 148.082 58.42 90)
 			(effects
@@
 			)
 		)
-		(property "Footprint" ""
+		(property "Footprint" "Button_Switch_SMD:SW_SPST_TL3342"
 			(at 193.04 83.82 0)
 			(effects
@@
 			)
 		)
-		(property "Footprint" ""
+		(property "Footprint" "gigalibrary:FSR402"
 			(at 184.912 58.42 90)
 			(effects
@@
 			)
 		)
-		(property "Footprint" ""
+		(property "Footprint" "gigalibrary:FSR402"
 			(at 127.762 58.42 90)
 			(effects
@@
 			)
 		)
-		(property "Footprint" ""
+		(property "Footprint" "Button_Switch_SMD:SW_SPST_TL3342"
 			(at 209.55 83.82 0)
 			(effects
@@
 			)
 		)
-		(property "Value" "~"
+		(property "Value" "Reset"
 			(at 21.082 22.606 0)
 			(effects
@@
 			)
 		)
-		(property "Footprint" ""
+		(property "Footprint" "Button_Switch_SMD:SW_SP3T_PCM13"
 			(at 27.94 31.75 0)
 			(effects

Commit message: hw: Finished footprints
Parts:
- removed J1: Conn_01x04_Socket, Connector_PinHeader_2.54mm:PinHeader_1x04_P2.54mm_Vertical, symbol Connector:Conn_01x04_Socket
- removed J2: Conn_01x05_Socket, gigalibrary:Joycon-FPC-1x05-P0.5mm, symbol Connector:Conn_01x05_Socket
- removed J3: Conn_01x05_Socket, Connector_PinHeader_2.54mm:PinHeader_1x04_P2.54mm_Vertical, symbol Connector:Conn_01x05_Socket
- added J1: Conn_01x05_Socket_FPC_Joycon, gigalibrary:Joycon-FPC-1x05-P0.5mm, symbol gigasound:Conn_01x05_Socket_FPC_Joycon
- added J2: Conn_01x05_Socket_UART, Connector_PinHeader_2.54mm:PinHeader_1x05_P2.54mm_Vertical, symbol gigasound:Conn_01x05_Socket_UART
- added J6: Conn_01x04_Socket_OLED, gigalibrary:PinSocket_1x04_P2.54mm_Vertical_OLED_0.96inch, symbol gigasound:Conn_01x04_Socket_OLED
- SW2: footprint Button_Switch_SMD:SW_SP3T_PCM13 -> Button_Switch_SMD:SW_Push_SPST_NO_Alps_SKRK
Connections:
- net 3.3V: now also J1.VCC, J6.VCC
- net ADC_CH14: now also J1.U/D
- net ADC_CH15: now also J1.L/R
- net GND: now also J1.GND, J2.1 (GND), J6.GND
- net RX: now also J2.3 (RX)
- net SCL: now also J6.SCL
- net SDA: now also J6.SDA
- net SWCLK: now also J2.5 (SWCLK)
- net SWDIO: now also J2.4 (SWDIO)
- net TX: now also J2.2 (TX)
Changed lines of the file:
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@@
 	)
 	(symbol
+		(lib_id "gigasound:Conn_01x05_Socket_FPC_Joycon")
+		(at 121.92 143.51 0)
+		(unit 1)
+		(exclude_from_sim no)
+		(in_bom yes)
+		(on_board yes)
+		(dnp no)
+		(fields_autoplaced yes)
+		(property "Reference" "J1"
+			(at 123.19 142.2399 0)
+			(effects
+				(font
+					(size 1.27 1.27)
+				)
+				(justify left)
+			)
+		)
+		(property "Value" "Conn_01x05_Socket_FPC_Joycon"
+			(at 123.19 144.7799 0)
+			(effects
+				(font
+					(size 1.27 1.27)
+				)
+				(justify left)
+			)
+		)
+		(property "Footprint" "gigalibrary:Joycon-FPC-1x05-P0.5mm"
+			(at 121.92 143.51 0)
+			(effects
+				(font
+					(size 1.27 1.27)
+				)
+				(hide yes)
+			)
+		)
+		(property "Datasheet" "~"
+			(at 121.92 143.51 0)
+			(effects
+				(font
+					(size 1.27 1.27)
+				)
+				(hide yes)
+			)
+		)
+		(property "Description" "Generic connector, single row, 01x05, script generated"
+			(at 121.92 143.51 0)
+			(effects
+				(font
+					(size 1.27 1.27)
+				)
+				(hide yes)
+			)
+		)
+		(pin "U/D"
+		)
+		(pin "BTN"
+		)
+		(pin "VCC"
+		)
+		(pin "GND"
+		)
+		(pin "L/R"
+		)
+		(instances
+			(project ""
+				(path "/8926df81-91df-4835-b346-b30b02cc5690"
+					(reference "J1")
+					(unit 1)
+				)
+			)
+		)
+	)
+	(symbol
 		(lib_id "power:VCC")
 		(at 201.93 39.37 0)
@@
 	)
 	(symbol
-		(lib_id "Connector:Conn_01x05_Socket")
-		(at 121.92 143.51 0)
+		(lib_id "power:VCC")
+		(at 110.49 161.29 90)
 		(unit 1)
 		(exclude_from_sim no)
@@
 		(on_board yes)
 		(dnp no)
-		(property "Reference" "J2"
-			(at 123.19 142.2399 0)
+		(fields_autoplaced yes)
+		(property "Reference" "#PWR028"
+			(at 114.3 161.29 0)
 			(effects
 				(font
 					(size 1.27 1.27)
 				)
-				(justify left)
+				(hide yes)
 			)
 		)
-		(property "Value" "Conn_01x05_Socket"
-			(at 123.19 144.526 0)
+		(property "Value" "3.3V"
+			(at 106.68 161.2899 90)
 			(effects
 				(font
@@
 			)
 		)
-		(property "Footprint" "gigalibrary:Joycon-FPC-1x05-P0.5mm"
-			(at 121.92 143.51 0)
+		(property "Footprint" ""
+			(at 110.49 161.29 0)
 			(effects
 				(font
@@
 			)
 		)
-		(property "Datasheet" "~"
-			(at 121.92 143.51 0)
+		(property "Datasheet" ""
+			(at 110.49 161.29 0)
 			(effects
 				(font
@@
 			)
 		)
-		(property "Description" "Generic connector, single row, 01x05, script generated"
-			(at 121.92 143.51 0)
+		(property "Description" "Power symbol creates a global label with name \"VCC\""
+			(at 110.49 161.29 0)
 			(effects
 				(font
@@
 			)
 		)
-		(pin "GND"
-		)
-		(pin "VCC"
-		)
-		(pin "U/D"
-		)
-		(pin "BTN"
-		)
-		(pin "L/R"
+		(pin "1"
 		)
 		(instances
 			(project "gigasound-hw"
 				(path "/8926df81-91df-4835-b346-b30b02cc5690"
-					(reference "J2")
+					(reference "#PWR028")
 					(unit 1)
 				)
@@
 	)
 	(symbol
-		(lib_id "power:VCC")
-		(at 110.49 161.29 90)
+		(lib_id "gigasound:Conn_01x04_Socket_OLED")
+		(at 121.92 161.29 0)
 		(unit 1)
 		(exclude_from_sim no)
@@
 		(dnp no)
 		(fields_autoplaced yes)
-		(property "Reference" "#PWR028"
-			(at 114.3 161.29 0)
+		(property "Reference" "J6"
+			(at 123.19 161.2899 0)
 			(effects
 				(font
 					(size 1.27 1.27)
 				)
-				(hide yes)
+				(justify left)
 			)
 		)
-		(property "Value" "3.3V"
-			(at 106.68 161.2899 90)
+		(property "Value" "Conn_01x04_Socket_OLED"
+			(at 123.19 163.8299 0)
 			(effects
 				(font
@@
 			)
 		)
-		(property "Footprint" ""
-			(at 110.49 161.29 0)
+		(property "Footprint" "gigalibrary:PinSocket_1x04_P2.54mm_Vertical_OLED_0.96inch"
+			(at 121.92 161.29 0)
 			(effects
 				(font
@@
 			)
 		)
-		(property "Datasheet" ""
-			(at 110.49 161.29 0)
+		(property "Datasheet" "~"
+			(at 121.92 161.29 0)
 			(effects
 				(font
@@
 			)
 		)
-		(property "Description" "Power symbol creates a global label with name \"VCC\""
-			(at 110.49 161.29 0)
+		(property "Description" "Generic connector, single row, 01x04, script generated"
+			(at 121.92 161.29 0)
 			(effects
 				(font
@@
 			)
 		)
-		(pin "1"
+		(pin "SDA"
+		)
+		(pin "GND"
+		)
+		(pin "VCC"
+		)
+		(pin "SCL"
 		)
 		(instances
-			(project "gigasound-hw"
+			(project ""
 				(path "/8926df81-91df-4835-b346-b30b02cc5690"
-					(reference "#PWR028")
+					(reference "J6")
 					(unit 1)
 				)
@@
 	)
 	(symbol
+		(lib_id "gigasound:Conn_01x05_Socket_UART")
+		(at 121.92 182.88 0)
+		(unit 1)
+		(exclude_from_sim no)
+		(in_bom yes)
+		(on_board yes)
+		(dnp no)
+		(fields_autoplaced yes)
+		(property "Reference" "J2"
+			(at 123.19 181.6099 0)
+			(effects
+				(font
+					(size 1.27 1.27)
+				)
+				(justify left)
+			)
+		)
+		(property "Value" "Conn_01x05_Socket_UART"
+			(at 123.19 184.1499 0)
+			(effects
+				(font
+					(size 1.27 1.27)
+				)
+				(justify left)
+			)
+		)
+		(property "Footprint" "Connector_PinHeader_2.54mm:PinHeader_1x05_P2.54mm_Vertical"
+			(at 121.92 182.88 0)
+			(effects
+				(font
+					(size 1.27 1.27)
+				)
+				(hide yes)
+			)
+		)
+		(property "Datasheet" "~"
+			(at 121.92 182.88 0)
+			(effects
+				(font
+					(size 1.27 1.27)
+				)
+				(hide yes)
+			)
+		)
+		(property "Description" "Generic connector, single row, 01x05, script generated"
+			(at 121.92 182.88 0)
+			(effects
+				(font
+					(size 1.27 1.27)
+				)
+				(hide yes)
+			)
+		)
+		(pin "2"
+		)
+		(pin "1"
+		)
+		(pin "3"
+		)
+		(pin "4"
+		)
+		(pin "5"
+		)
+		(instances
+			(project ""
+				(path "/8926df81-91df-4835-b346-b30b02cc5690"
+					(reference "J2")
+					(unit 1)
+				)
+			)
+		)
+	)
+	(symbol
 		(lib_id "Device:C")
 		(at 191.77 129.54 0)
@@
 	)
 	(symbol
-		(lib_name "Conn_01x05_Socket_1")
-		(lib_id "Connector:Conn_01x05_Socket")
-		(at 121.92 182.88 0)
-		(unit 1)
-		(exclude_from_sim no)
-		(in_bom yes)
-		(on_board yes)
-		(dnp no)
-		(fields_autoplaced yes)
-		(property "Reference" "J3"
-			(at 123.19 181.6099 0)
-			(effects
-				(font
-					(size 1.27 1.27)
-				)
-				(justify left)
-			)
-		)
-		(property "Value" "Conn_01x05_Socket"
-			(at 123.19 184.1499 0)
-			(effects
-				(font
-					(size 1.27 1.27)
-				)
-				(justify left)
-			)
-		)
-		(property "Footprint" "Connector_PinHeader_2.54mm:PinHeader_1x04_P2.54mm_Vertical"
-			(at 121.92 182.88 0)
-			(effects
-				(font
-					(size 1.27 1.27)
-				)
-				(hide yes)
-			)
-		)
-		(property "Datasheet" "~"
-			(at 121.92 182.88 0)
-			(effects
-				(font
-					(size 1.27 1.27)
-				)
-				(hide yes)
-			)
-		)
-		(property "Description" "Generic connector, single row, 01x05, script generated"
-			(at 121.92 182.88 0)
-			(effects
-				(font
-					(size 1.27 1.27)
-				)
-				(hide yes)
-			)
-		)
-		(pin "SWCLK"
-		)
-		(pin "RX"
-		)
-		(pin "GND"
-		)
-		(pin "SWDIO"
-		)
-		(pin "TX"
-		)
-		(instances
-			(project "gigasound-hw"
-				(path "/8926df81-91df-4835-b346-b30b02cc5690"
-					(reference "J3")
-					(unit 1)
-				)
-			)
-		)
-	)
-	(symbol
 		(lib_id "power:GND")
 		(at 64.77 138.43 0)
@@
 	)
 	(symbol
-		(lib_id "Connector:Conn_01x04_Socket")
-		(at 121.92 161.29 0)
-		(unit 1)
-		(exclude_from_sim no)
-		(in_bom yes)
-		(on_board yes)
-		(dnp no)
-		(fields_autoplaced yes)
-		(property "Reference" "J1"
-			(at 123.19 161.2899 0)
-			(effects
-				(font
-					(size 1.27 1.27)
-				)
-				(justify left)
-			)
-		)
-		(property "Value" "Conn_01x04_Socket"
-			(at 123.19 163.8299 0)
-			(effects
-				(font
-					(size 1.27 1.27)
-				)
-				(justify left)
-			)
-		)
-		(property "Footprint" "Connector_PinHeader_2.54mm:PinHeader_1x04_P2.54mm_Vertical"
-			(at 121.92 161.29 0)
-			(effects
-				(font
-					(size 1.27 1.27)
-				)
-				(hide yes)
-			)
-		)
-		(property "Datasheet" "~"
-			(at 121.92 161.29 0)
-			(effects
-				(font
-					(size 1.27 1.27)
-				)
-				(hide yes)
-			)
-		)
-		(property "Description" "Generic connector, single row, 01x04, script generated"
-			(at 121.92 161.29 0)
-			(effects
-				(font
-					(size 1.27 1.27)
-				)
-				(hide yes)
-			)
-		)
-		(pin "GND"
-		)
-		(pin "SDA"
-		)
-		(pin "SCL"
-		)
-		(pin "VCC"
-		)
-		(instances
-			(project "gigasound-hw"
-				(path "/8926df81-91df-4835-b346-b30b02cc5690"
-					(reference "J1")
-					(unit 1)
-				)
-			)
-		)
-	)
-	(symbol
 		(lib_id "Switch:SW_Push")
 		(at 198.12 83.82 90)
@@
 			)
 		)
-		(property "Footprint" "Button_Switch_SMD:SW_SP3T_PCM13"
+		(property "Footprint" "Button_Switch_SMD:SW_Push_SPST_NO_Alps_SKRK"
 			(at 27.94 31.75 0)
 			(effects

Commit message: hw: finish layout
Parts:
- Y1: symbol Device:Crystal -> Device:Crystal_GND24
Connections:
- net ADC_CH0: now also U1.23 (PA7); no longer U1.14 (PA0)
- net ADC_CH1: now also U1.22 (PA6); no longer U1.15 (PA1)
- net ADC_CH2: now also U1.21 (PA5); no longer U1.16 (PA2)
- net ADC_CH3: now also U1.20 (PA4); no longer U1.17 (PA3)
- net ADC_CH4: now also U1.17 (PA3); no longer U1.20 (PA4)
- net ADC_CH5: now also U1.14 (PA0); no longer U1.21 (PA5)
- net ADC_CH6: now also U1.15 (PA1); no longer U1.22 (PA6)
- net ADC_CH7: now also U1.16 (PA2); no longer U1.23 (PA7)
- net GND: now also Y1.2, Y1.4
- net OSC_IN: now also Y1.3; no longer Y1.2
- net USB_DM renamed USB_D-
- net USB_DP renamed USB_D+

Commit message: hw: start routing
Connections:
- net LED_play_pause_mode/LED_OUT renamed LED_5050x8/LED_OUT
Changed lines of the file:
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@@
 	)
 	(junction
+		(at 271.78 21.59)
+		(diameter 0)
+		(color 0 0 0 0)
+	)
+	(junction
 		(at 19.05 36.83)
 		(diameter 0)
@@
 	(wire
 		(pts
-			(xy 52.07 30.48) (xy 52.07 31.75)
+			(xy 265.43 21.59) (xy 271.78 21.59)
 		)
 		(stroke
@@
 	(wire
 		(pts
-			(xy 271.78 21.59) (xy 267.97 21.59)
+			(xy 52.07 30.48) (xy 52.07 31.75)
 		)
 		(stroke
@@
 	(wire
 		(pts
+			(xy 238.76 21.59) (xy 243.84 21.59)
+		)
+		(stroke
+			(width 0)
+			(type default)
+		)
+	)
+	(wire
+		(pts
 			(xy 109.22 166.37) (xy 116.84 166.37)
 		)
@@
 	(wire
 		(pts
+			(xy 271.78 21.59) (xy 273.05 21.59)
+		)
+		(stroke
+			(width 0)
+			(type default)
+		)
+	)
+	(wire
+		(pts
 			(xy 168.91 54.61) (xy 173.99 54.61)
 		)
@@
 	(wire
 		(pts
-			(xy 236.22 21.59) (xy 243.84 21.59)
-		)
-		(stroke
-			(width 0)
-			(type default)
-		)
-	)
-	(wire
-		(pts
 			(xy 31.75 111.76) (xy 31.75 110.49)
 		)
@@
 	(wire
 		(pts
-			(xy 170.18 21.59) (xy 179.07 21.59)
+			(xy 170.18 21.59) (xy 182.88 21.59)
 		)
 		(stroke
@@
 	(wire
 		(pts
-			(xy 200.66 21.59) (xy 209.55 21.59)
+			(xy 209.55 21.59) (xy 214.63 21.59)
 		)
 		(stroke
@@
 	)
 	(sheet
-		(at 209.55 19.05)
+		(at 182.88 19.05)
 		(size 26.67 5.08)
 		(exclude_from_sim no)
@@
 		)
 		(property "Sheetname" "LED_2020_Trimmer"
-			(at 209.55 18.3384 0)
+			(at 182.88 18.3384 0)
 			(effects
 				(font
@@
 		)
 		(property "Sheetfile" "led_trimmer.kicad_sch"
-			(at 209.55 24.7146 0)
+			(at 182.88 24.7146 0)
 			(effects
 				(font
@@
 		)
 		(pin "LED_IN" input
-			(at 209.55 21.59 180)
+			(at 182.88 21.59 180)
 			(effects
 				(font
@@
 		)
 		(pin "LED_OUT" output
-			(at 236.22 21.59 0)
+			(at 209.55 21.59 0)
 			(effects
 				(font
@@
 	)
 	(sheet
-		(at 243.84 19.05)
+		(at 214.63 19.05)
 		(size 24.13 5.08)
 		(exclude_from_sim no)
@@
 		)
 		(property "Sheetname" "LED_play_pause_mode"
-			(at 243.84 18.3384 0)
+			(at 214.63 18.3384 0)
 			(effects
 				(font
@@
 		)
 		(property "Sheetfile" "led_play_pausa_mode.kicad_sch"
-			(at 243.84 24.7146 0)
+			(at 214.63 24.7146 0)
 			(effects
 				(font
@@
 		)
 		(pin "LED_IN" input
-			(at 243.84 21.59 180)
+			(at 214.63 21.59 180)
 			(effects
 				(font
@@
 		)
 		(pin "LED_OUT" output
-			(at 267.97 21.59 0)
+			(at 238.76 21.59 0)
 			(effects
 				(font
@@
 	)
 	(sheet
-		(at 179.07 19.05)
+		(at 243.84 19.05)
 		(size 21.59 5.08)
 		(exclude_from_sim no)
@@
 		)
 		(property "Sheetname" "LED_5050x8"
-			(at 179.07 18.3384 0)
+			(at 243.84 18.3384 0)
 			(effects
 				(font
@@
 		)
 		(property "Sheetfile" "led5050x8.kicad_sch"
-			(at 179.07 24.7146 0)
+			(at 243.84 24.7146 0)
 			(effects
 				(font
@@
 		)
 		(pin "LED_IN" input
-			(at 179.07 21.59 180)
+			(at 243.84 21.59 180)
 			(effects
 				(font
@@
 		)
 		(pin "LED_OUT" output
-			(at 200.66 21.59 0)
+			(at 265.43 21.59 0)
 			(effects
 				(font

Commit message: hw: added esd protection and caps
Parts:
- added C34, C35, C36, C37, C38, C39, C40, C41, C42: DNF, Capacitor_SMD:C_0402_1005Metric_Pad0.74x0.62mm_HandSolder, symbol Device:C
- added U2: USBLC6-2SC6, Package_TO_SOT_SMD:SOT-23-6, symbol Power_Protection:USBLC6-2SC6
Connections:
- net 5V: now also U2.5 (VBUS)
- net ADC_CH0: now also C34.2
- net ADC_CH1: now also C35.2
- net ADC_CH2: now also C36.2
- net ADC_CH3: now also C37.2
- net ADC_CH4: now also C38.2
- net ADC_CH5: now also C39.2
- net ADC_CH6: now also C40.2
- net ADC_CH7: now also C41.2
- net ADC_CH8: now also C42.2
- net GND: now also C34.1, C35.1, C36.1, C37.1, C38.1, C39.1, C40.1, C41.1, C42.1, U2.2 (GND)
- net USB_D+: now also U2.4 (I/O2); no longer J4.A6 (D+), J4.B6 (D+)
- net USB_D-: now also U2.6 (I/O1); no longer J4.A7 (D-), J4.B7 (D-)
- new net: J4.A7 (D-), J4.B7 (D-), U2.1 (I/O1)
- new net: J4.A6 (D+), J4.B6 (D+), U2.3 (I/O2)
Other:
- moved on the sheet: R7, R8, RV1

Commit message: hw: final touches
Parts:
- J5: footprint Connector_PinHeader_1.00mm:PinHeader_1x01_P1.00mm_Vertical -> Connector_PinHeader_2.54mm:PinHeader_1x03_P2.54mm_Vertical; symbol Connector:Conn_01x01_Socket -> Connector:Conn_01x03_Socket
Connections:
- net 5V: now also J5.1 (Pin_1)
- net GND: now also J5.3 (Pin_3)
- net LED_5050x8/LED_OUT: now also J5.2 (Pin_2); no longer J5.1 (Pin_1)
Changed lines of the file:
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@@
 	(text "LED"
 		(exclude_from_sim no)
-		(at 276.86 17.272 0)
+		(at 172.974 16.764 0)
 		(effects
 			(font
@@
 	)
 	(junction
-		(at 271.78 21.59)
-		(diameter 0)
-		(color 0 0 0 0)
-	)
-	(junction
 		(at 19.05 36.83)
 		(diameter 0)
@@
 	(wire
 		(pts
-			(xy 265.43 21.59) (xy 271.78 21.59)
-		)
-		(stroke
-			(width 0)
-			(type default)
-		)
-	)
-	(wire
-		(pts
 			(xy 52.07 30.48) (xy 52.07 31.75)
 		)
@@
 	(wire
 		(pts
-			(xy 271.78 21.59) (xy 273.05 21.59)
-		)
-		(stroke
-			(width 0)
-			(type default)
-		)
-	)
-	(wire
-		(pts
 			(xy 168.91 53.34) (xy 173.99 53.34)
 		)
@@
 	(wire
 		(pts
+			(xy 265.43 21.59) (xy 273.05 21.59)
+		)
+		(stroke
+			(width 0)
+			(type default)
+		)
+	)
+	(wire
+		(pts
 			(xy 72.39 39.37) (xy 86.36 39.37)
 		)
@@
 	)
 	(symbol
-		(lib_id "Connector:Conn_01x01_Socket")
-		(at 276.86 21.59 0)
+		(lib_id "Connector:Conn_01x03_Socket")
+		(at 278.13 21.59 0)
 		(unit 1)
 		(exclude_from_sim no)
@@
 		(dnp no)
 		(property "Reference" "J5"
-			(at 278.13 20.3199 0)
+			(at 279.146 18.288 0)
 			(effects
 				(font
@@
 		)
 		(property "Value" "PIN_LED_OUT"
-			(at 268.478 23.114 0)
+			(at 278.892 21.844 0)
 			(effects
 				(font
@@
 			)
 		)
-		(property "Footprint" "Connector_PinHeader_1.00mm:PinHeader_1x01_P1.00mm_Vertical"
-			(at 276.86 21.59 0)
+		(property "Footprint" "Connector_PinHeader_2.54mm:PinHeader_1x03_P2.54mm_Vertical"
+			(at 278.13 21.59 0)
 			(effects
 				(font
@@
 		)
 		(property "Datasheet" "~"
-			(at 276.86 21.59 0)
+			(at 278.13 21.59 0)
 			(effects
 				(font
@@
 			)
 		)
-		(property "Description" "Generic connector, single row, 01x01, script generated"
-			(at 276.86 21.59 0)
+		(property "Description" "Generic connector, single row, 01x03, script generated"
+			(at 278.13 21.59 0)
 			(effects
 				(font
@@
 		(pin "1"
 		)
+		(pin "2"
+		)
+		(pin "3"
+		)
 		(instances
 			(project ""
@@
 	)
 	(symbol
+		(lib_id "power:GND")
+		(at 273.05 24.13 0)
+		(unit 1)
+		(exclude_from_sim no)
+		(in_bom yes)
+		(on_board yes)
+		(dnp no)
+		(fields_autoplaced yes)
+		(property "Reference" "#PWR060"
+			(at 273.05 30.48 0)
+			(effects
+				(font
+					(size 1.27 1.27)
+				)
+				(hide yes)
+			)
+		)
+		(property "Value" "GND"
+			(at 273.05 29.21 0)
+			(effects
+				(font
+					(size 1.27 1.27)
+				)
+			)
+		)
+		(property "Footprint" ""
+			(at 273.05 24.13 0)
+			(effects
+				(font
+					(size 1.27 1.27)
+				)
+				(hide yes)
+			)
+		)
+		(property "Datasheet" ""
+			(at 273.05 24.13 0)
+			(effects
+				(font
+					(size 1.27 1.27)
+				)
+				(hide yes)
+			)
+		)
+		(property "Description" "Power symbol creates a global label with name \"GND\" , ground"
+			(at 273.05 24.13 0)
+			(effects
+				(font
+					(size 1.27 1.27)
+				)
+				(hide yes)
+			)
+		)
+		(pin "1"
+		)
+		(instances
+			(project ""
+				(path "/8926df81-91df-4835-b346-b30b02cc5690"
+					(reference "#PWR060")
+					(unit 1)
+				)
+			)
+		)
+	)
+	(symbol
 		(lib_id "Connector:TestPoint")
 		(at 72.39 87.63 270)
@@
 					(unit 1)
 				)
+			)
+		)
+	)
+	(symbol
+		(lib_id "power:VCC")
+		(at 273.05 19.05 0)
+		(unit 1)
+		(exclude_from_sim no)
+		(in_bom yes)
+		(on_board yes)
+		(dnp no)
+		(property "Reference" "#PWR061"
+			(at 273.05 22.86 0)
+			(effects
+				(font
+					(size 1.27 1.27)
+				)
+				(hide yes)
+			)
+		)
+		(property "Value" "5V"
+			(at 273.05 15.748 0)
+			(effects
+				(font
+					(size 1.27 1.27)
+				)
+			)
+		)
+		(property "Footprint" ""
+			(at 273.05 19.05 0)
+			(effects
+				(font
+					(size 1.27 1.27)
+				)
+				(hide yes)
+			)
+		)
+		(property "Datasheet" ""
+			(at 273.05 19.05 0)
+			(effects
+				(font
+					(size 1.27 1.27)
+				)
+				(hide yes)
+			)
+		)
+		(property "Description" "Power symbol creates a global label with name \"VCC\""
+			(at 273.05 19.05 0)
+			(effects
+				(font
+					(size 1.27 1.27)
+				)
+				(hide yes)
+			)
+		)
+		(pin "1"
+		)
+		(instances
+			(project "gigasound-hw"
+				(path "/8926df81-91df-4835-b346-b30b02cc5690"
+					(reference "#PWR061")
+					(unit 1)
+				)
