File: gigasound-hw/gigasound-hw.kicad_sch (KiCad schematic)
At the start: 87 parts, among them J1 Conn_01x05_Socket_FPC_Joycon, J2 Conn_01x05_Socket_UART, J4 USB_C_Receptacle_USB2.0_16P, J5 PIN_LED_OUT, J6 Conn_01x04_Socket_OLED, SW1 PLAY, SW2 Reset, SW4 STOP, SW5 MODE, U1 STM32F401RETx, U2 USBLC6-2SC6, U5 AMS1117-3.3, Y1 12MHz

Commit message: fix clock
Parts:
- removed C11: 100nF, Capacitor_SMD:C_0402_1005Metric_Pad0.74x0.62mm_HandSolder, symbol Device:C
Connections:
- net GND: now also U1.12 (VSSA)
- net VDDA: no longer U1.12 (VSSA)
Changed lines of the file:
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@@
 	)
 	(junction
+		(at 54.61 128.27)
+		(diameter 0)
+		(color 0 0 0 0)
+	)
+	(junction
 		(at 186.69 64.77)
 		(diameter 0)
@@
 	)
 	(junction
-		(at 64.77 128.27)
-		(diameter 0)
-		(color 0 0 0 0)
-	)
-	(junction
 		(at 214.63 96.52)
 		(diameter 0)
@@
 	(wire
 		(pts
+			(xy 54.61 128.27) (xy 57.15 128.27)
+		)
+		(stroke
+			(width 0)
+			(type default)
+		)
+	)
+	(wire
+		(pts
 			(xy 24.13 29.21) (xy 19.05 29.21)
 		)
@@
 	(wire
 		(pts
-			(xy 64.77 128.27) (xy 64.77 127)
-		)
-		(stroke
-			(width 0)
-			(type default)
-		)
-	)
-	(wire
-		(pts
 			(xy 59.69 31.75) (xy 59.69 30.48)
 		)
@@
 	(wire
 		(pts
-			(xy 57.15 128.27) (xy 64.77 128.27)
-		)
-		(stroke
-			(width 0)
-			(type default)
-		)
-	)
-	(wire
-		(pts
 			(xy 149.86 62.23) (xy 149.86 64.77)
 		)
@@
 	(wire
 		(pts
+			(xy 54.61 128.27) (xy 54.61 130.81)
+		)
+		(stroke
+			(width 0)
+			(type default)
+		)
+	)
+	(wire
+		(pts
 			(xy 191.77 124.46) (xy 191.77 121.92)
 		)
@@
 	(wire
 		(pts
-			(xy 54.61 125.73) (xy 54.61 130.81)
+			(xy 54.61 125.73) (xy 54.61 128.27)
 		)
 		(stroke
@@
 	(wire
 		(pts
-			(xy 64.77 138.43) (xy 64.77 135.89)
-		)
-		(stroke
-			(width 0)
-			(type default)
-		)
-	)
-	(wire
-		(pts
 			(xy 36.83 36.83) (xy 33.02 36.83)
 		)
@@
 	)
 	(symbol
-		(lib_id "power:VDD")
-		(at 64.77 127 0)
-		(unit 1)
-		(exclude_from_sim no)
-		(in_bom yes)
-		(on_board yes)
-		(dnp no)
-		(property "Reference" "#PWR014"
-			(at 64.77 130.81 0)
-			(effects
-				(font
-					(size 1.27 1.27)
-				)
-				(hide yes)
-			)
-		)
-		(property "Value" "VDDA"
-			(at 64.008 126.238 0)
-			(effects
-				(font
-					(size 1.27 1.27)
-				)
-				(justify right)
-			)
-		)
-		(property "Footprint" ""
-			(at 64.77 127 0)
-			(effects
-				(font
-					(size 1.27 1.27)
-				)
-				(hide yes)
-			)
-		)
-		(property "Datasheet" ""
-			(at 64.77 127 0)
-			(effects
-				(font
-					(size 1.27 1.27)
-				)
-				(hide yes)
-			)
-		)
-		(property "Description" "Power symbol creates a global label with name \"VDD\""
-			(at 64.77 127 0)
-			(effects
-				(font
-					(size 1.27 1.27)
-				)
-				(hide yes)
-			)
-		)
-		(pin "1"
-		)
-		(instances
-			(project ""
-				(path "/8926df81-91df-4835-b346-b30b02cc5690"
-					(reference "#PWR014")
-					(unit 1)
-				)
-			)
-		)
-	)
-	(symbol
 		(lib_id "power:GND")
 		(at 173.99 134.62 0)
@@
 					(unit 1)
 				)
-			)
-		)
-	)
-	(symbol
-		(lib_id "Device:C")
-		(at 64.77 132.08 180)
-		(unit 1)
-		(exclude_from_sim no)
-		(in_bom yes)
-		(on_board yes)
-		(dnp no)
-		(property "Reference" "C11"
-			(at 61.468 130.048 90)
-			(effects
-				(font
-					(size 1.27 1.27)
-				)
-				(justify left)
-			)
-		)
-		(property "Value" "100nF"
-			(at 68.326 129.032 90)
-			(effects
-				(font
-					(size 1.27 1.27)
-				)
-				(justify left)
-			)
-		)
-		(property "Footprint" "Capacitor_SMD:C_0402_1005Metric_Pad0.74x0.62mm_HandSolder"
-			(at 63.8048 128.27 0)
-			(effects
-				(font
-					(size 1.27 1.27)
-				)
-				(hide yes)
-			)
-		)
-		(property "Datasheet" "~"
-			(at 64.77 132.08 0)
-			(effects
-				(font
-					(size 1.27 1.27)
-				)
-				(hide yes)
-			)
-		)
-		(property "Description" "Unpolarized capacitor"
-			(at 64.77 132.08 0)
-			(effects
-				(font
-					(size 1.27 1.27)
-				)
-				(hide yes)
-			)
-		)
-		(pin "1"
-		)
-		(pin "2"
-		)
-		(instances
-			(project ""
-				(path "/8926df81-91df-4835-b346-b30b02cc5690"
-					(reference "C11")
-					(unit 1)
-				)
