File: gigasound-hw/gigasound-hw.kicad_sch (KiCad schematic)
At the start: 86 parts, among them J1 Conn_01x05_Socket_FPC_Joycon, J2 Conn_01x05_Socket_UART, J4 USB_C_Receptacle_USB2.0_16P, J5 PIN_LED_OUT, J6 Conn_01x04_Socket_OLED, SW1 PLAY, SW2 Reset, SW4 STOP, SW5 MODE, U1 STM32F401RETx, U2 USBLC6-2SC6, U5 AMS1117-3.3, Y1 12MHz

Commit message: hw: fix big mistake
Parts:
- added C11: 100nF, Capacitor_SMD:C_0402_1005Metric_Pad0.74x0.62mm_HandSolder, symbol Device:C
Connections:
- net GND: now also C11.2
- net VDDA: now also C11.1
Changed lines of the file:
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@@
 	)
 	(junction
+		(at 64.77 137.16)
+		(diameter 0)
+		(color 0 0 0 0)
+	)
+	(junction
 		(at 19.05 40.64)
 		(diameter 0)
@@
 	)
 	(junction
-		(at 54.61 128.27)
-		(diameter 0)
-		(color 0 0 0 0)
-	)
-	(junction
 		(at 186.69 64.77)
 		(diameter 0)
@@
 	(wire
 		(pts
-			(xy 54.61 128.27) (xy 57.15 128.27)
-		)
-		(stroke
-			(width 0)
-			(type default)
-		)
-	)
-	(wire
-		(pts
 			(xy 24.13 29.21) (xy 19.05 29.21)
 		)
@@
 	(wire
 		(pts
+			(xy 64.77 137.16) (xy 64.77 138.43)
+		)
+		(stroke
+			(width 0)
+			(type default)
+		)
+	)
+	(wire
+		(pts
 			(xy 245.11 41.91) (xy 265.43 41.91)
 		)
@@
 	(wire
 		(pts
-			(xy 54.61 128.27) (xy 54.61 130.81)
+			(xy 54.61 125.73) (xy 54.61 130.81)
 		)
 		(stroke
@@
 	(wire
 		(pts
-			(xy 57.15 125.73) (xy 57.15 128.27)
+			(xy 57.15 125.73) (xy 57.15 137.16)
 		)
 		(stroke
@@
 	(wire
 		(pts
-			(xy 54.61 125.73) (xy 54.61 128.27)
-		)
-		(stroke
-			(width 0)
-			(type default)
-		)
-	)
-	(wire
-		(pts
 			(xy 181.61 74.93) (xy 181.61 78.74)
 		)
@@
 	(wire
 		(pts
+			(xy 57.15 137.16) (xy 64.77 137.16)
+		)
+		(stroke
+			(width 0)
+			(type default)
+		)
+	)
+	(wire
+		(pts
 			(xy 104.14 146.05) (xy 116.84 146.05)
 		)
@@
 	)
 	(symbol
+		(lib_id "power:VDDA")
+		(at 64.77 129.54 0)
+		(unit 1)
+		(exclude_from_sim no)
+		(in_bom yes)
+		(on_board yes)
+		(dnp no)
+		(property "Reference" "#PWR014"
+			(at 64.77 133.35 0)
+			(effects
+				(font
+					(size 1.27 1.27)
+				)
+				(hide yes)
+			)
+		)
+		(property "Value" "VDDA"
+			(at 66.802 125.984 0)
+			(effects
+				(font
+					(size 1.27 1.27)
+				)
+			)
+		)
+		(property "Footprint" ""
+			(at 64.77 129.54 0)
+			(effects
+				(font
+					(size 1.27 1.27)
+				)
+				(hide yes)
+			)
+		)
+		(property "Datasheet" ""
+			(at 64.77 129.54 0)
+			(effects
+				(font
+					(size 1.27 1.27)
+				)
+				(hide yes)
+			)
+		)
+		(property "Description" "Power symbol creates a global label with name \"VDDA\""
+			(at 64.77 129.54 0)
+			(effects
+				(font
+					(size 1.27 1.27)
+				)
+				(hide yes)
+			)
+		)
+		(pin "1"
+		)
+		(instances
+			(project "gigasound-hw"
+				(path "/8926df81-91df-4835-b346-b30b02cc5690"
+					(reference "#PWR014")
+					(unit 1)
+				)
+			)
+		)
+	)
+	(symbol
 		(lib_id "Device:C")
 		(at 144.78 58.42 180)
@@
 					(unit 1)
 				)
+			)
+		)
+	)
+	(symbol
+		(lib_id "Device:C")
+		(at 64.77 133.35 0)
+		(unit 1)
+		(exclude_from_sim no)
+		(in_bom yes)
+		(on_board yes)
+		(dnp no)
+		(property "Reference" "C11"
+			(at 58.166 133.604 0)
+			(effects
+				(font
+					(size 1.27 1.27)
+				)
+				(justify left)
+			)
+		)
+		(property "Value" "100nF"
+			(at 67.564 134.112 0)
+			(effects
+				(font
+					(size 1.27 1.27)
+				)
+				(justify left)
+			)
+		)
+		(property "Footprint" "Capacitor_SMD:C_0402_1005Metric_Pad0.74x0.62mm_HandSolder"
+			(at 65.7352 137.16 0)
+			(effects
+				(font
+					(size 1.27 1.27)
+				)
+				(hide yes)
+			)
+		)
+		(property "Datasheet" "~"
+			(at 64.77 133.35 0)
+			(effects
+				(font
+					(size 1.27 1.27)
+				)
+				(hide yes)
+			)
+		)
+		(property "Description" "Unpolarized capacitor"
+			(at 64.77 133.35 0)
+			(effects
+				(font
+					(size 1.27 1.27)
+				)
+				(hide yes)
+			)
+		)
+		(pin "2"
+		)
+		(pin "1"
+		)
+		(instances
+			(project "gigasound-hw"
+				(path "/8926df81-91df-4835-b346-b30b02cc5690"
+					(reference "C11")
+					(unit 1)
+				)

Commit message: hw: new pcb revision candidate
Connections:
- net ADC_CH0: now also C39.2, R18.2, R19.1, U1.14 (PA0); no longer C34.2, R1.1, R3.2, U1.23 (PA7)
- net ADC_CH1: now also C40.2, R20.2, R21.1, U1.15 (PA1); no longer C35.2, R11.1, R9.2, U1.22 (PA6)
- net ADC_CH2: now also C41.2, R22.2, R23.1, U1.16 (PA2); no longer C36.2, R12.2, R13.1, U1.21 (PA5)
- net ADC_CH3: now also C38.2, R16.2, R17.1, U1.17 (PA3); no longer C37.2, R14.2, R15.1, U1.20 (PA4)
- net ADC_CH4: now also C37.2, R14.2, R15.1, U1.20 (PA4); no longer C38.2, R16.2, R17.1, U1.17 (PA3)
- net ADC_CH5: now also C36.2, R12.2, R13.1, U1.21 (PA5); no longer C39.2, R18.2, R19.1, U1.14 (PA0)
- net ADC_CH6: now also C35.2, R11.1, R9.2, U1.22 (PA6); no longer C40.2, R20.2, R21.1, U1.15 (PA1)
- net ADC_CH7: now also C34.2, R1.1, R3.2, U1.23 (PA7); no longer C41.2, R22.2, R23.1, U1.16 (PA2)
Changed lines of the file:
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@@
 		)
 	)
-	(label "ADC_CH0"
+	(label "ADC_CH7"
 		(at 135.89 53.34 0)
 		(effects
@@
 		)
 	)
-	(label "ADC_CH1"
+	(label "ADC_CH6"
 		(at 86.36 54.61 0)
 		(effects
@@
 		)
 	)
-	(label "ADC_CH7"
+	(label "ADC_CH2"
 		(at 86.36 44.45 180)
 		(effects
@@
 		)
 	)
-	(label "ADC_CH2"
+	(label "ADC_CH5"
 		(at 86.36 52.07 0)
 		(effects
@@
 		)
 	)
-	(label "ADC_CH1"
+	(label "ADC_CH6"
 		(at 154.94 53.34 0)
 		(effects
@@
 		)
 	)
+	(label "ADC_CH2"
+		(at 270.51 53.34 0)
+		(effects
+			(font
+				(size 1.27 1.27)
+			)
+			(justify left bottom)
+		)
+	)
 	(label "ADC_CH7"
-		(at 270.51 53.34 0)
-		(effects
-			(font
-				(size 1.27 1.27)
-			)
-			(justify left bottom)
-		)
-	)
-	(label "ADC_CH0"
 		(at 86.36 57.15 0)
 		(effects
@@
 		)
 	)
-	(label "ADC_CH6"
+	(label "ADC_CH1"
 		(at 86.36 41.91 180)
 		(effects
@@
 		)
 	)
-	(label "ADC_CH4"
+	(label "ADC_CH3"
 		(at 212.09 53.34 0)
 		(effects
@@
 		)
 	)
-	(label "ADC_CH2"
+	(label "ADC_CH5"
 		(at 173.99 53.34 0)
 		(effects
@@
 		)
 	)
-	(label "ADC_CH4"
+	(label "ADC_CH3"
 		(at 86.36 46.99 0)
 		(effects
@@
 		)
 	)
-	(label "ADC_CH5"
+	(label "ADC_CH0"
 		(at 86.36 39.37 180)
 		(effects
@@
 		)
 	)
-	(label "ADC_CH3"
+	(label "ADC_CH4"
 		(at 86.36 49.53 0)
 		(effects
@@
 		)
 	)
-	(label "ADC_CH6"
+	(label "ADC_CH1"
 		(at 250.19 54.61 0)
 		(effects
@@
 		)
 	)
-	(label "ADC_CH3"
+	(label "ADC_CH4"
 		(at 191.77 53.34 0)
 		(effects
@@
 		)
 	)
-	(label "ADC_CH5"
+	(label "ADC_CH0"
 		(at 231.14 53.34 0)
 		(effects
